File: thumbstick/thumbstick.kicad_sch (KiCad schematic)
At the start: 2 parts, among them P1 rkjxv1220001

Commit message: Thubmstick v1
Parts:
- removed P1: rkjxv1220001, rkjxv1220001:rkjxv1220001, symbol rkjxv1220001:rkjxv1220001
- removed out1: Conn_01x04_Female, Connector_PinSocket_2.54mm:PinSocket_1x04_P2.54mm_Vertical_SMD_Pin1Left, symbol Connector:Conn_01x04_Female
- added C1: 10uF, Capacitor_SMD:C_0603_1608Metric, symbol Device:C_Small
- added C2, C3: 100nF, Capacitor_SMD:C_0603_1608Metric, symbol Device:C_Small
- added H1: Conn_01x05, Connector_Molex:Molex_PicoBlade_53047-0510_1x05_P1.25mm_Vertical, symbol Connector_Generic:Conn_01x05
- added MNT1: MountingHole, MountingHole:MountingHole_2.2mm_M2_Pad, symbol Mechanical:MountingHole
- added POT1: RKJXV122400R, rkjxv1220001:RKJXV122400R, symbol rkjxv1220001:RKJXV122400R
Connections:
- net GND: now also C1.2, C2.2, C3.2, H1.5 (Pin_5), POT1.3, POT1.6, POT1.7
- net VCC: now also C1.1, C2.1, C3.1, H1.1 (Pin_1), POT1.1, POT1.4
- new net P_OUT: H1.4 (Pin_4), POT1.8
- new net X_OUT: H1.2 (Pin_2), POT1.2
- new net Y_OUT: H1.3 (Pin_3), POT1.5
- no-connect marks 0 -> 1
Other:
- company: (none) -> Diego Covarrubias
- title: (none) -> Keeb Stick
