File: host/host.kicad_sch (KiCad schematic)
At the start: 22 parts

Commit message: host v1
Parts:
- removed H? (x2): Conn_01x06, symbol Connector_Generic:Conn_01x06
- removed H?: Conn_01x40, symbol Connector_Generic:Conn_01x40
- added C11, C12: 20p, Capacitor_SMD:C_0603_1608Metric, symbol Device:C_Small
- added H1: MountingHole, MountingHole:MountingHole_2.2mm_M2_Pad, symbol Mechanical:MountingHole
- added J1: Conn_01x02, Connector_Molex:Molex_PicoBlade_53047-0210_1x02_P1.25mm_Vertical, symbol Connector_Generic:Conn_01x02
- added J3, J4: Conn_01x05, Connector_Molex:Molex_PicoBlade_53047-0510_1x05_P1.25mm_Vertical, symbol Connector_Generic:Conn_01x05
- added R1: 33K, Resistor_SMD:R_0603_1608Metric, symbol Device:R_Small
- added R2: 82K, Resistor_SMD:R_0603_1608Metric, symbol Device:R_Small
- added R3: 0, Resistor_SMD:R_0603_1608Metric, symbol Device:R_Small
- added SW2: SW_SPST, KLIB:ALPS_SKRKAEE020, symbol Switch:SW_SPST
- added U2: USBLC6-2SC6, Package_TO_SOT_SMD:SOT-23-6, symbol Power_Protection:USBLC6-2SC6
- added Y1: 8M, Crystal:Crystal_SMD_5032-2Pin_5.0x3.2mm, symbol Device:Crystal_Small
- C1, C2, C3, C9: renamed from C?; value 10uF -> 10u; footprint (none) -> Capacitor_SMD:C_0603_1608Metric
- C10, C14, C4, C5, C6, C7, C8: renamed from C?; value 100nF -> 100n; footprint (none) -> Capacitor_SMD:C_0603_1608Metric
- C13: renamed from C?; value 4.7uF -> 4.7u; footprint (none) -> Capacitor_SMD:C_0603_1608Metric
- FB1: renamed from FB?; value 120R -> 120; footprint (none) -> Inductor_SMD:L_0603_1608Metric
- J2: renamed from USB1; footprint (none) -> KLIB:JST_UBA-4R-D14T-4D
- R4, R5: renamed from R?; value 10k -> 10K; footprint (none) -> Resistor_SMD:R_0603_1608Metric
- SW1: renamed from SW?; footprint (none) -> KLIB:ALPS_SSSS912000
- renumbered LDO1 to U1, MCU1 to U3
Connections:
- net BOOT0: now also R4.2; no longer R4.1
- net BOOT1: now also R5.2; no longer R5.1
- net GND: now also C11.2, C12.2, J1.2 (Pin_2), R2.2, SW2.2 (B), U2.2 (GND); no longer R5.2
- net HSE_IN: now also C11.1, Y1.1
- net HSE_OUT: now also R3.1
- net RAW_USB_D+: now also U2.3 (I/O2)
- net RAW_USB_D-: now also U2.1 (I/O1)
- net USB_D+: now also U2.4 (I/O2)
- net USB_D-: now also U2.6 (I/O1)
- net at SW1.2 (B): now also R4.1; no longer R4.2
- net CN_MISO renamed MISO_L
- net MISO_L: now also J3.3 (Pin_3)
- net CN_MOSI renamed MOSI_L
- net MOSI_L: now also J3.2 (Pin_2)
- net CN_NSS renamed NSS_L
- net NSS_L: now also J3.5 (Pin_5)
- net CN_SCK renamed SCK_L
- net SCK_L: now also J3.4 (Pin_4)
- net DS_BLPWM: no longer names the net of U3.14 (PA0)
- net DS_D0: no longer names the net of U3.9 (PC1)
- net DS_D1: no longer names the net of U3.10 (PC2)
- net DS_D10: no longer names the net of U3.38 (PC7)
- net DS_D11: no longer names the net of U3.37 (PC6)
- net DS_D12: no longer names the net of U3.36 (PB15)
- net DS_D13: no longer names the net of U3.35 (PB14)
- net DS_D14: no longer names the net of U3.34 (PB13)
- net DS_D15: no longer names the net of U3.33 (PB12)
- net DS_D2: no longer names the net of U3.25 (PC5)
- net DS_D3: no longer names the net of U3.26 (PB0)
- net DS_D4: no longer names the net of U3.27 (PB1)
- net DS_D5: no longer names the net of U3.29 (PB10)
- net DS_D6 renamed USB_VBUS
- net USB_VBUS: now also R1.2, R2.1
- net DS_D7: no longer names the net of U3.41 (PA8)
- net DS_D8: no longer names the net of U3.40 (PC9)
- net DS_D9: no longer names the net of U3.39 (PC8)
- net EXT_MISO renamed MISO_R
- net MISO_R: now also J4.3 (Pin_3)
- net EXT_MOSI renamed MOSI_R
- net MOSI_R: now also J4.2 (Pin_2)
- net EXT_NSS renamed NSS_R
- net NSS_R: now also J4.5 (Pin_5)
- net EXT_SCK renamed SCK_R
- net SCK_R: now also J4.4 (Pin_4)
- net NC_PA1: no longer names the net of U3.15 (PA1)
- net NC_PA10: no longer names the net of U3.43 (PA10)
- net NC_PA13: no longer names the net of U3.46 (PA13)
- net NC_PA14: no longer names the net of U3.49 (PA14)
- net NC_PA2: no longer names the net of U3.16 (PA2)
- net NC_PA3: no longer names the net of U3.17 (PA3)
- net NC_PB3: no longer names the net of U3.55 (PB3)
- net NC_PB4: no longer names the net of U3.56 (PB4)
- net NC_PB5: no longer names the net of U3.57 (PB5)
- net NC_PB6: no longer names the net of U3.58 (PB6)
- net NC_PB7: no longer names the net of U3.59 (PB7)
- net NC_PB8: no longer names the net of U3.61 (PB8)
- net NC_PB9: no longer names the net of U3.62 (PB9)
- net NC_PC0: no longer names the net of U3.8 (PC0)
- net NC_PC13: no longer names the net of U3.2 (PC13)
- net NC_PC14: no longer names the net of U3.3 (PC14)
- net NC_PC15: no longer names the net of U3.4 (PC15)
- net NC_PC3: no longer names the net of U3.11 (PC3)
- net NC_PC4 renamed MSC_R
- net MSC_R: now also J4.1 (Pin_1)
- net NC_PD2 renamed MSC_L
- net MSC_L: now also J3.1 (Pin_1)
- net USB_BUS renamed RAW_USB_VBUS
- net RAW_USB_VBUS: now also R1.1, U2.5 (VBUS)
- net VBUS renamed 5V
- net 5V: now also J1.1 (Pin_1)
- new net: R5.1, SW2.1 (A)
- new net: C12.1, R3.2, Y1.2
- no-connect marks 8 -> 35
Other:
- note added: "BOARD MOUNT"
- note added: "BOOT"
- note added: "Controller-Controller SPI"
- note added: "MCU"
- note added: "PWR"
- note added: "USB"
- note added: "XTAL, VCAP, NRST"
- company: (none) -> Diego Covarrubias
- title: (none) -> Keeb Host
- moved on the sheet: C1, C10, C13, C14, C2, C3, C4, C5, C6, C7, C8, C9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
