File: host/host.kicad_sch (KiCad schematic)
At the start: 31 parts, among them J1 Conn_01x02, J2 USB_A, J3 Conn_01x05, J4 Conn_01x05, SW1 SW_SPDT, SW2 SW_SPST, U1 AP2127N-3.3, U2 USBLC6-2SC6, U3 STM32F401RCT6, Y1 8M

Commit message: power v1, updated host to v2
Parts:
- removed J2: USB_A, KLIB:JST_UBA-4R-D14T-4D, symbol Connector:USB_A
- removed J3, J4: Conn_01x05, Connector_Molex:Molex_PicoBlade_53047-0510_1x05_P1.25mm_Vertical, symbol Connector_Generic:Conn_01x05
- removed SW2: SW_SPST, KLIB:ALPS_SKRKAEE020, symbol Switch:SW_SPST
- added J2: USB_C_Receptacle_USB2.0, Connector_USB:USB_C_Receptacle_HRO_TYPE-C-31-M-12, symbol Connector:USB_C_Receptacle_USB2.0
- added J3, J4: Conn_01x04, Connector_Molex:Molex_PicoBlade_53047-0410_1x04_P1.25mm_Vertical, symbol Connector_Generic:Conn_01x04
- added R6, R7: 5.1K, Resistor_SMD:R_0603_1608Metric, symbol Device:R_Small
- J1: footprint Connector_Molex:Molex_PicoBlade_53047-0210_1x02_P1.25mm_Vertical -> klib:MOLEX_533750210-Mini-Lock-2Pin-Through-Hole
- R4: renamed from R1; value 33K -> 48K
- R5: renamed from R2; value 82K -> 72K
- SW1: footprint KLIB:ALPS_SSSS912000 -> klib:ALPS_SSSS912000
- renumbered R3 to R1, R4 to R2, R5 to R3
Connections:
- net RAW_USB_VBUS is gone; now on net USB_VBUS: R4.1, U2.5 (VBUS)
- net 5V: now also J1.2 (Pin_2); no longer J1.1 (Pin_1)
- net GND: now also J1.1 (Pin_1), R3.1, J2.A1 (GND), J2.A12 (GND), J2.B1 (GND), J2.B12 (GND), J2.S1 (SHIELD), R6.2, R7.2; no longer J1.2 (Pin_2)
- net MISO_L: now also J3.2 (Pin_2)
- net MISO_R: now also J4.2 (Pin_2)
- net MOSI_L: now also J3.1 (Pin_1)
- net MOSI_R: now also J4.1 (Pin_1)
- net NSS_L: now also J3.4 (Pin_4)
- net NSS_R: now also J4.4 (Pin_4)
- net SCK_L: now also J3.3 (Pin_3)
- net SCK_R: now also J4.3 (Pin_3)
- net USB_VBUS: now also J2.A4 (VBUS), J2.A9 (VBUS), J2.B4 (VBUS), J2.B9 (VBUS); no longer R4.2, R5.1, U3.42 (PA9)
- net MSC_L: no longer names the net of U3.54 (PD2)
- net MSC_R: no longer names the net of U3.24 (PC4)
- net RAW_USB_D+ renamed USB_RAW_D+
- net USB_RAW_D+: now also J2.A6 (D+), J2.B6 (D+)
- net RAW_USB_D- renamed USB_RAW_D-
- net USB_RAW_D-: now also J2.A7 (D-), J2.B7 (D-)
- new net USB_CC1: J2.A5 (CC1), R6.1
- new net USB_CC2: J2.B5 (CC2), R7.1
- new net USB_VBUS_SIG: R4.2, R5.1, U3.42 (PA9)
- no-connect marks 35 -> 38
Other:
- note added: "5V -> 3V3"
- note added: "Controller <-> Controller"
- note added: "MOUNT"
- note added: "PWR IN"
- note added: "VDD"
- note added: "VDDA"
- note removed: "BOARD MOUNT"
- note removed: "Controller-Controller SPI"
- moved on the sheet: C1, C10, C11, C12, C13, C14, C2, C3, C4, C5, C6, C7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

Commit message: update controller and host boards
Parts:
- renumbered U3 to U2, U2 to U3
Changed lines of the file:
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@@
   (symbol (lib_id "MCU_ST_STM32F4:STM32F401RCTx") (at 61.976 202.184 0) (unit 1)
     (in_bom yes) (on_board yes)
-    (property "Reference" "U3" (id 0) (at 69.088 158.242 0)
+    (property "Reference" "U2" (id 0) (at 69.088 158.242 0)
       (effects (font (size 1 1)) (justify left))
     )
@@
   (symbol (lib_id "Power_Protection:USBLC6-2SC6") (at 204.47 217.17 0) (unit 1)
     (in_bom yes) (on_board yes)
-    (property "Reference" "U2" (id 0) (at 207.264 206.502 0)
+    (property "Reference" "U3" (id 0) (at 207.264 206.502 0)
       (effects (font (size 1 1)) (justify left))
     )
@@
       (reference "U1") (unit 1) (value "AP2127N-3.3") (footprint "Package_TO_SOT_SMD:SOT-23")
     )
+    (path "/0cf90a94-8a8c-402d-a846-a0a32251e41c"
+      (reference "U2") (unit 1) (value "STM32F401RCT6") (footprint "Package_QFP:LQFP-64_10x10mm_P0.5mm")
+    )
     (path "/46bf371d-1bf5-4b9f-a9d5-d73816ac87ae"
-      (reference "U2") (unit 1) (value "USBLC6-2SC6") (footprint "Package_TO_SOT_SMD:SOT-23-6")
-    )
-    (path "/0cf90a94-8a8c-402d-a846-a0a32251e41c"
-      (reference "U3") (unit 1) (value "STM32F401RCT6") (footprint "Package_QFP:LQFP-64_10x10mm_P0.5mm")
+      (reference "U3") (unit 1) (value "USBLC6-2SC6") (footprint "Package_TO_SOT_SMD:SOT-23-6")
     )
     (path "/7facd3ee-8f53-41cd-9607-37f24abf1516"
