File: power/power.kicad_sch (KiCad schematic)
At the start: 2 parts

Commit message: power v1, updated host to v2
Parts:
- removed J?: Conn_01x02, symbol Connector_Generic:Conn_01x02
- removed PS?: IRM-10-5, Converter_ACDC:Converter_ACDC_MeanWell_IRM-10-xx_THT, symbol Converter_ACDC:IRM-10-5
- added H1, H2: MountingHole, MountingHole:MountingHole_2.2mm_M2_Pad, symbol Mechanical:MountingHole
- added J1, J2: Screw_Terminal_01x01, klib:DORABO_DB136HA-10.16-1P, symbol Connector:Screw_Terminal_01x01
- added J3, J4, J5, J6, J7, J8: Conn_01x02, klib:MOLEX_533750210-Mini-Lock-2Pin-Through-Hole, symbol Connector_Generic:Conn_01x02
- added PS1: IRM-20-5, Converter_ACDC:Converter_ACDC_MeanWell_IRM-20-xx_THT, symbol Converter_ACDC:IRM-20-5
Connections:
- new net 5V: J3.1 (Pin_1), J4.1 (Pin_1), J5.1 (Pin_1), J6.2 (Pin_2), J7.2 (Pin_2), J8.2 (Pin_2), PS1.4 (+Vo)
- new net AC_L: J1.1 (Pin_1), PS1.1 (AC/L)
- new net AC_N: J2.1 (Pin_1), PS1.2 (AC/N)
- new net GND: J3.2 (Pin_2), J4.2 (Pin_2), J5.2 (Pin_2), J6.1 (Pin_1), J7.1 (Pin_1), J8.1 (Pin_1), PS1.3 (-Vo)
