File: controller/controller.kicad_sch (KiCad schematic)
At the start: 74 parts, among them SW1 SW_SPDT, SW2 SW_SPST

Commit message: Sensor v1
Changed lines of the file:
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@@
     (pin "9")
+  )
+  (symbol (lib_id "Regulator_Linear:AP2127N-3.3") (at 138.684 42.418 0) (unit 1)
+    (in_bom yes) (on_board yes) (fields_autoplaced)
+    (property "Reference" "LDO1" (id 0) (at 138.684 35.56 0))
+    (property "Value" "AP2127N-3.3" (id 1) (at 138.684 38.1 0))
+    (property "Footprint" "Package_TO_SOT_SMD:SOT-23" (id 2) (at 138.684 36.703 0)
+      (effects (font (size 1.27 1.27) italic) hide)
+    )
+    (property "Datasheet" "https://www.diodes.com/assets/Datasheets/AP2127.pdf" (id 3) (at 138.684 42.418 0)
+      (effects (font (size 1.27 1.27)) hide)
+    )
+    (pin "1")
+    (pin "2")
+    (pin "3")
   )
   (symbol (lib_id "Device:C_Small") (at 440.182 50.419 0) (unit 1)
@@
     (pin "6")
   )
-  (symbol (lib_id "Regulator_Linear:AP2127N-3.3") (at 138.684 42.418 0) (unit 1)
-    (in_bom yes) (on_board yes) (fields_autoplaced)
-    (property "Reference" "LDO1" (id 0) (at 138.684 36.83 0)
-      (effects (font (size 1 1)))
-    )
-    (property "Value" "AP2127N-3.3" (id 1) (at 138.684 39.37 0)
-      (effects (font (size 1 1) italic))
-    )
-    (property "Footprint" "Package_TO_SOT_SMD:SOT-23" (id 2) (at 138.684 36.703 0)
-      (effects (font (size 1.27 1.27) italic) hide)
-    )
-    (property "Datasheet" "https://www.diodes.com/assets/Datasheets/AP2127.pdf" (id 3) (at 138.684 42.418 0)
-      (effects (font (size 1.27 1.27)) hide)
-    )
-    (pin "1")
-    (pin "2")
-    (pin "3")
-  )
   (symbol (lib_id "Connector_Generic:Conn_01x05") (at 340.36 373.634 0) (unit 1)
     (in_bom yes) (on_board yes) (fields_autoplaced)
@@
       (reference "H14") (unit 1) (value "Conn_01x03") (footprint "Connector_Molex:Molex_PicoBlade_53047-0310_1x03_P1.25mm_Vertical")
     )
-    (path "/c43cde42-06c8-4a38-a840-be919d24617a"
+    (path "/082fbcf6-a43d-4e76-ba92-bf94710b0792"
       (reference "LDO1") (unit 1) (value "AP2127N-3.3") (footprint "Package_TO_SOT_SMD:SOT-23")
     )

Commit message: start work on host mcu
Parts:
- FB1: footprint Inductor_SMD:L_1206_3216Metric -> Inductor_SMD:L_0603_1608Metric
Changed lines of the file:
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@@
     (property "Reference" "FB1" (id 0) (at 316.0649 35.56 90))
     (property "Value" "120R" (id 1) (at 316.0649 38.1 90))
-    (property "Footprint" "Inductor_SMD:L_1206_3216Metric" (id 2) (at 316.103 43.942 90)
+    (property "Footprint" "Inductor_SMD:L_0603_1608Metric" (id 2) (at 316.103 43.942 90)
       (effects (font (size 1.27 1.27)) hide)
     )
@@
     )
     (path "/8b4289f2-9a86-4728-acfc-6857feae1132"
-      (reference "FB1") (unit 1) (value "120R") (footprint "Inductor_SMD:L_1206_3216Metric")
+      (reference "FB1") (unit 1) (value "120R") (footprint "Inductor_SMD:L_0603_1608Metric")
     )
     (path "/c36b3a61-3f93-4a26-bac4-d190cb007fea"

Commit message: update controller and host boards
Parts:
- removed H1, H2, H4, H5, H6: Conn_01x06, Connector_Molex:Molex_PicoBlade_53047-0610_1x06_P1.25mm_Vertical, symbol Connector_Generic:Conn_01x06
- removed H10, H11, H12, H13, H14: Conn_01x03, Connector_Molex:Molex_PicoBlade_53047-0310_1x03_P1.25mm_Vertical, symbol Connector_Generic:Conn_01x03
- removed H3, H8, H9: Conn_01x05, Connector_Molex:Molex_PicoBlade_53047-0510_1x05_P1.25mm_Vertical, symbol Connector_Generic:Conn_01x05
- removed H7: Conn_01x04, Connector_Molex:Molex_PicoBlade_53047-0410_1x04_P1.25mm_Vertical, symbol Connector_Generic:Conn_01x04
- removed LDO1: AP2127N-3.3, Package_TO_SOT_SMD:SOT-23, symbol Regulator_Linear:AP2127N-3.3
- removed R10, R11, R12, R13, R14, R15, R16, R17, R18, R19, R20, R21, R22, R23, R24, R25, R26, R27, R28, R29, R5, R6, R7, R8, R9: 10KR, Resistor_SMD:R_0603_1608Metric, symbol Device:R_Small
- removed SW2: SW_SPST, Custom:ALPS_SKRKAEE020, symbol Switch:SW_SPST
- removed USB1: USB_A, Custom:JST_UBA-4R-D14T-4D, symbol Connector:USB_A
- removed XTAL1: 8MHz, Crystal:Crystal_SMD_5032-2Pin_5.0x3.2mm, symbol Device:Crystal_Small
- added J1, J11, J3: Conn_01x02, klib:MOLEX_533750210-Mini-Lock-2Pin-Through-Hole, symbol Connector_Generic:Conn_01x02
- added J10, J4, J7, J8, J9: Conn_01x05, Connector_Molex:Molex_PicoBlade_53047-0510_1x05_P1.25mm_Vertical, symbol Connector_Generic:Conn_01x05
- added J2: USB_C_Receptacle_USB2.0, Connector_USB:USB_C_Receptacle_HRO_TYPE-C-31-M-12, symbol Connector:USB_C_Receptacle_USB2.0
- added J5, J6: Conn_01x04, Connector_Molex:Molex_PicoBlade_53047-0410_1x04_P1.25mm_Vertical, symbol Connector_Generic:Conn_01x04
- added U1: AP2127N-3.3, Package_TO_SOT_SMD:SOT-23, symbol Regulator_Linear:AP2127N-3.3
- added Y1: 8M, Crystal:Crystal_SMD_5032-2Pin_5.0x3.2mm, symbol Device:Crystal_Small
- C1, C2, C3, C9: value 10uF -> 10u
- C10, C15, C16, C17, C18, C19, C20, C21, C4, C5, C6, C7, C8: value 100nF -> 100n
- C11: value 4.7uF -> 20p
- C12: value 100nF -> 20p
- C13: value 20pF -> 4.7u
- C14: value 20pF -> 100n
- R1: value 0R -> 0
- R2, R3, R4: value 10KR -> 10K
- SW1: footprint Custom:ALPS_SSSS912000 -> klib:ALPS_SSSS912000
- renumbered MNT1 to H1, MCU1 to U2, ESD1 to U3, VT1 to U4
Connections:
- net KP1 is gone; now on net LED4: U2.57 (PB5)
- net KP2 is gone; now on net LED3: U2.58 (PB6)
- net KP3 is gone; now on net LED2: U2.59 (PB7)
- net KR1 is gone; now on net GND: R3.2
- net KT1_IN is gone; now on net ST_P: R4.2
- net KT2 is gone; now on net LED_OE: U2.55 (PB3)
- net BOOT0: now also R2.2; no longer R2.1
- net GND: now also C12.2, C20.2, C21.2, J1.1 (Pin_1), J10.5 (Pin_5), J11.2 (Pin_2), J2.A1 (GND), J2.A12 (GND), J2.B1 (GND), J2.B12 (GND), J2.S1 (SHIELD), J3.2 (Pin_2), J9.1 (Pin_1), U1.1 (GND); no longer C12.1, C20.1, C21.1
- net HSE_IN: now also C11.1, Y1.1; no longer C13.1
- net HSE_OUT: now also R1.1; no longer R1.2
- net LED1_OUT: now also J4.1 (Pin_1)
- net LED2: no longer U2.62 (PB9)
- net LED2_OUT: now also J4.2 (Pin_2)
- net LED3: now also U4.5 (A4); no longer U2.2 (PC13), U4.4 (A3)
- net LED3_OUT: now also U4.16 (B4), J4.3 (Pin_3); no longer U4.17 (B3)
- net LED4: now also U4.7 (A6); no longer U2.3 (PC14), U4.5 (A4)
- net LED4_OUT: now also U4.14 (B6), J4.4 (Pin_4); no longer U4.16 (B4)
- net LED5: now also U2.56 (PB4), U4.9 (A8); no longer U2.8 (PC0), U4.6 (A5)
- net LED5_OUT: now also U4.12 (B8), J4.5 (Pin_5); no longer U4.15 (B5)
- net LED_OE: no longer U2.9 (PC1)
- net NRST: now also C14.1; no longer C12.2
- net ST_P: now also U2.14 (PA0); no longer U2.15 (PA1)
- net ST_P_IN: now also R4.1, J10.4 (Pin_4)
- net ST_X: now also C20.1, U2.16 (PA2), J10.2 (Pin_2); no longer C15.1, U2.17 (PA3)
- net ST_Y: now also C21.1, U2.15 (PA1), J10.3 (Pin_3); no longer C16.1, U2.16 (PA2)
- net TR1: now also U2.10 (PC2), J9.4 (Pin_4); no longer U2.14 (PA0)
- net TR2: now also U2.9 (PC1), J9.3 (Pin_3); no longer U2.11 (PC3)
- net TR3: now also U2.8 (PC0), J9.2 (Pin_2); no longer U2.10 (PC2)
- net USB_RAW_D+: now also J2.A6 (D+), J2.B6 (D+)
- net USB_RAW_D-: now also J2.A7 (D-), J2.B7 (D-)
- net VCAP: now also C13.1; no longer C11.1
- net at SW1.2 (B): now also R2.1; no longer R2.2
- net +3.3VA renamed VREF
- net +3V3 renamed 3V3
- net 3V3: now also C15.1, J10.1 (Pin_1), J9.5 (Pin_5), U1.2 (VO); no longer C20.2
- net BOOT1/KR1 renamed BOOT1
- net CN_MISO renamed MISO_R
- net MISO_R: now also J6.2 (Pin_2)
- net CN_MOSI renamed MOSI_R
- net MOSI_R: now also J6.1 (Pin_1)
- net CN_NSS renamed NSS_R
- net NSS_R: now also J6.4 (Pin_4)
- net CN_SCK renamed SCK_R
- net SCK_R: now also J6.3 (Pin_3)
- net KI1 renamed COL5
- net COL5: now also J7.1 (Pin_1)
- net KI2 renamed COL4
- net COL4: now also J7.2 (Pin_2)
- net KI3 renamed COL3
- net COL3: now also J7.3 (Pin_3)
- net KI4 renamed COL2
- net COL2: now also J7.4 (Pin_4)
- net KI5 renamed COL1
- net COL1: now also J7.5 (Pin_5)
- net KM1 renamed ROW1
- net ROW1: now also J8.1 (Pin_1)
- net KM2 renamed ROW2
- net ROW2: now also J8.2 (Pin_2)
- net KM3 renamed ROW3
- net ROW3: now also J8.3 (Pin_3)
- net KM4 renamed ROW4
- net ROW4: now also J8.4 (Pin_4)
- net KM5 renamed ROW5
- net ROW5: now also J8.5 (Pin_5)
- net KR2: no longer names the net of U2.27 (PB1)
- net KR3: no longer names the net of U2.26 (PB0)
- net KR4: no longer names the net of U2.25 (PC5)
- net KR5: no longer names the net of U2.24 (PC4)
- removed net KT1: R4.1, U2.56 (PB4)
- net KT3: no longer names the net of U2.54 (PD2)
- net KT4: no longer names the net of U2.49 (PA14)
- net NC_PA10: no longer names the net of U2.43 (PA10)
- net NC_PA13 renamed USB_HPS
- net USB_HPS: now also J2.A8 (SBU1), J2.B8 (SBU2)
- net NC_PB10: no longer names the net of U2.29 (PB10)
- net NC_PC15: no longer names the net of U2.4 (PC15)
- net SN_MISO renamed MISO_L
- net MISO_L: now also J5.2 (Pin_2)
- net SN_MOSI renamed MOSI_L
- net MOSI_L: now also J5.1 (Pin_1)
- net SN_NSS renamed NSS_L
- net NSS_L: now also J5.4 (Pin_4)
- net SN_SCK renamed SCK_L
- net SCK_L: now also J5.3 (Pin_3)
- net VBUS renamed 5V
- net 5V: now also C16.1, J1.2 (Pin_2), J11.1 (Pin_1), J2.A4 (VBUS), J2.A9 (VBUS), J2.B4 (VBUS), J2.B9 (VBUS), J3.1 (Pin_1), U1.3 (VI); no longer C21.2
- new net: C12.1, R1.2, Y1.2
- no-connect marks 7 -> 22
Other:
- note added: "Controller <-> Controller"
- note added: "Key Matrix"
- note added: "LED"
- note added: "PWR"
- note added: "Sensor PWR"
- note added: "Stick"
- note added: "Trigger"
- note added: "XTAL, VCAP, NRST"
- note removed: "CONNECTORS"
- note removed: "HSE"
- note removed: "KI (Index Keys)"
- note removed: "KM (Middle Keys)"
- note removed: "KP (Pinky Keys)"
- note removed: "KR (Ring Keys)"
- note removed: "KR1 shares a 10KR with BOOT1 (See BOOT section)"
- note removed: "KT (Thumb Keys)"
- note removed: "LED IO Translation"
- note removed: "MCU_VBUS"
- note removed: "MCU_VDD"
- note removed: "MCU_VDDA"
- note removed: "NC"
- note removed: "NRST"
- note removed: "ST"
- note removed: "TR"
- note removed: "VCAP"
- moved on the sheet: H1, U2, U3, U4
